Commit message: reorganized urdf into description subpackage

File: boris_description/urdf/boris_description.urdf (robot description, URDF)
Before this commit: robot boris, 9 links, 8 joints
Links:
- link arm_link: geometry collision mesh filename=package://boris_description/meshes/arm_link.STL; visual mesh filename=package://boris_description/meshes/arm_link.STL
- link base_link: geometry collision mesh filename=package://boris_description/meshes/base_link.STL; visual mesh filename=package://boris_description/meshes/base_link.STL
- link camera_link: geometry collision mesh filename=package://boris_description/meshes/camera_link.STL; visual mesh filename=package://boris_description/meshes/camera_link.STL
- link camera_tilt_link: geometry collision mesh filename=package://boris_description/meshes/camera_tilt_link.STL; visual mesh filename=package://boris_description/meshes/camera_tilt_link.STL
- link camera_yaw_link: geometry collision mesh filename=package://boris_description/meshes/camera_yaw_link.STL; visual mesh filename=package://boris_description/meshes/camera_yaw_link.STL
- link elbow_link: geometry collision mesh filename=package://boris_description/meshes/elbow_link.STL; visual mesh filename=package://boris_description/meshes/elbow_link.STL
- link left_wheel_link: geometry collision mesh filename=package://boris_description/meshes/left_wheel_link.STL; visual mesh filename=package://boris_description/meshes/left_wheel_link.STL
- link right_wheel_link: geometry collision mesh filename=package://boris_description/meshes/right_wheel_link.STL; visual mesh filename=package://boris_description/meshes/right_wheel_link.STL
- link shoulder_link: geometry collision mesh filename=package://boris_description/meshes/shoulder_link.STL; visual mesh filename=package://boris_description/meshes/shoulder_link.STL

Commit message: fixed camera gimbal joint names

File: boris_description/urdf/boris_description.urdf (robot description, URDF)
Before this commit: robot boris_description, 9 links, 8 joints
Joints:
- removed joint camera_yaw_ioint
- added joint camera_yaw_joint: type continuous, parent base_link, child camera_yaw_link, origin xyz=0 -0.10927 1.1284 rpy=1.5708 0 -1.4442, axis 0 -1 0

Commit message: working camera code + scan but no output

File: boris_description/urdf/boris_description.urdf (robot description, URDF)
Before this commit: robot boris_description, 9 links, 8 joints
Joints:
- joint camera_joint: origin xyz=0.05255 -0.006823 -0.01495 rpy=-3.1416 0 -3.1416 -> xyz=0 0 0 rpy=0 1.57079632679 1.57079632679

Commit message: new urdf for testing

File: boris_description/urdf/boris_description.urdf (robot description, URDF)
Before this commit: robot boris_description, 9 links, 8 joints
Links:
- removed link arm_link
- removed link camera_link
- removed link elbow_link
- removed link shoulder_link
- added link camera, mass 0.0447521989519099; collision mesh filename=package://boris_description/meshes/camera.STL; visual mesh filename=package://boris_description/meshes/camera.STL
- added link gps_link, mass 0.00832308173444994; collision mesh filename=package://boris_description/meshes/gps_link.STL; visual mesh filename=package://boris_description/meshes/gps_link.STL
- added link imu, mass 0.000983130183652036; collision mesh filename=package://boris_description/meshes/imu.STL; visual mesh filename=package://boris_description/meshes/imu.STL
- link base_link: mass None -> 6.25092338139406
- link camera_tilt_link: mass 0.0136650343598071 -> 0.0136650343598073
- link camera_yaw_link: mass 0.011452 -> 0.0236989643956742
- link left_wheel_link: mass 0.95801 -> 0.958008587347379
- link right_wheel_link: mass 0.95801 -> 0.958008587347378
Joints:
- removed joint arm_joint
- removed joint elbow_joint
- removed joint shoulder_joint
- added joint gps_joint: type fixed, parent base_link, child gps_link, origin xyz=0.026225 -0.24281 1.1433 rpy=0 0 3.1416, axis 0 0 0
- added joint imu_joint: type fixed, parent base_link, child imu, origin xyz=0.013335 -0.212040199999975 0.20085 rpy=1.5707963267949 0 3.14159265358979, axis 0 0 0
- joint camera_joint: child camera_link -> camera; origin xyz=0 0 0 rpy=0 1.57079632679 1.57079632679 -> xyz=0.041323 -0.035823 -0.01495 rpy=3.1416 0 0
- joint camera_tilt_joint: origin xyz=0 -0.043915 0.013263 rpy=0.03975 1.5708 0 -> xyz=0.041323 0.061915 0 rpy=0 0 3.1416
- joint camera_yaw_joint: axis 0 -1 0 -> 0 1 0; origin xyz=0 -0.10927 1.1284 rpy=1.5708 0 -1.4442 -> xyz=0 -0.16095 1.1464 rpy=-1.5708 0 3.1416

Commit message: updated urdf with realsense ros package camera model

File: boris_description/urdf/boris_description.urdf (robot description, URDF)
Before this commit: robot boris_description, 8 links, 7 joints
Links:
- removed link camera
- added link camera_bottom_screw_frame
- added link camera_color_frame
- added link camera_color_optical_frame
- added link camera_depth_frame
- added link camera_depth_optical_frame
- added link camera_infra1_frame
- added link camera_infra1_optical_frame
- added link camera_infra2_frame
- added link camera_infra2_optical_frame
- added link camera_link, mass 0.564; collision box size=0.02505 0.09 0.025; visual mesh filename=package://boris_description/meshes/d435.dae
Joints:
- added joint camera_color_joint: type fixed, parent camera_link, child camera_color_frame, origin xyz=0 0.015 0 rpy=0 0 0
- added joint camera_color_optical_joint: type fixed, parent camera_color_frame, child camera_color_optical_frame, origin xyz=0 0 0 rpy=-1.57079632679 0 -1.57079632679
- added joint camera_depth_joint: type fixed, parent camera_link, child camera_depth_frame, origin xyz=0 0 0 rpy=0 0 0
- added joint camera_depth_optical_joint: type fixed, parent camera_depth_frame, child camera_depth_optical_frame, origin xyz=0 0 0 rpy=-1.57079632679 0 -1.57079632679
- added joint camera_infra1_joint: type fixed, parent camera_link, child camera_infra1_frame, origin xyz=0 0.0 0 rpy=0 0 0
- added joint camera_infra1_optical_joint: type fixed, parent camera_infra1_frame, child camera_infra1_optical_frame, origin xyz=0 0 0 rpy=-1.57079632679 0 -1.57079632679
- added joint camera_infra2_joint: type fixed, parent camera_link, child camera_infra2_frame, origin xyz=0 -0.05 0 rpy=0 0 0
- added joint camera_infra2_optical_joint: type fixed, parent camera_infra2_frame, child camera_infra2_optical_frame, origin xyz=0 0 0 rpy=-1.57079632679 0 -1.57079632679
- added joint camera_link_joint: type fixed, parent camera_bottom_screw_frame, child camera_link, origin xyz=0 0.0175 0.0125 rpy=0 0 0
- joint camera_joint: child camera -> camera_bottom_screw_frame

Commit message: major working update, urdf fixed/updated, working gmapping except planar, working gimbal, other improvements

File: boris_description/urdf/boris_description.urdf (robot description, URDF)
Before this commit: robot boris_description, 17 links, 16 joints
Joints:
- joint camera_joint: origin xyz=0.041323 -0.035823 -0.01495 rpy=3.1416 0 0 -> xyz=0.041323 -0.023823 0 rpy=3.1416 1.57079632679 1.57079632679

Commit message: fixed urdf base link orientation

File: boris_description/urdf/boris_description.urdf (robot description, URDF)
Before this commit: robot boris_description, 17 links, 16 joints
Links:
- link gps_link: mass 0.00832308173444994 -> 0.00810471227426635
- link right_wheel_link: mass 0.958008587347378 -> 0.958008587347379
Joints:
- joint camera_yaw_joint: origin xyz=0 -0.16095 1.1464 rpy=-1.5708 0 3.1416 -> xyz=-0.16095 0 1.1464 rpy=-1.5708 0 1.5708
- joint gps_joint: origin xyz=0.026225 -0.24281 1.1433 rpy=0 0 3.1416 -> xyz=-0.24281 -0.026225 1.1433 rpy=0 0 1.5708
- joint imu_joint: origin xyz=0.013335 -0.212040199999975 0.20085 rpy=1.5707963267949 0 3.14159265358979 -> xyz=-0.21204 -0.013335 0.20085 rpy=1.5708 0 1.5708
- joint left_wheel_joint: origin xyz=-0.3074 -1.02E-05 -0.017901 rpy=-3.1416 0 3.1416 -> xyz=-1.02E-05 0.3074 -0.017901 rpy=-3.1416 0 1.5708
- joint right_wheel_joint: origin xyz=0.3074 -1.02E-05 -0.017901 rpy=3.1416 0 0 -> xyz=-1.02E-05 -0.3074 -0.017901 rpy=3.1416 0 -1.5708

Commit message: urdf

File: boris_description/urdf/boris_description.urdf (robot description, URDF)
Before this commit: robot boris_description, 17 links, 16 joints
Links:
- added link camera2_bottom_screw_frame
- added link camera2_color_frame
- added link camera2_color_optical_frame
- added link camera2_depth_frame
- added link camera2_depth_optical_frame
- added link camera2_infra1_frame
- added link camera2_infra1_optical_frame
- added link camera2_infra2_frame
- added link camera2_infra2_optical_frame
- added link camera2_link, mass 0.564; collision box size=0.02505 0.09 0.025; visual mesh filename=package://boris_description/meshes/d435.dae
Joints:
- added joint camera2_color_joint: type fixed, parent camera2_link, child camera2_color_frame, origin xyz=0 0.015 0 rpy=0 0 0
- added joint camera2_color_optical_joint: type fixed, parent camera2_color_frame, child camera2_color_optical_frame, origin xyz=0 0 0 rpy=-1.57079632679 0 -1.57079632679
- added joint camera2_depth_joint: type fixed, parent camera2_link, child camera2_depth_frame, origin xyz=0 0 0 rpy=0 0 0
- added joint camera2_depth_optical_joint: type fixed, parent camera2_depth_frame, child camera2_depth_optical_frame, origin xyz=0 0 0 rpy=-1.57079632679 0 -1.57079632679
- added joint camera2_infra1_joint: type fixed, parent camera2_link, child camera2_infra1_frame, origin xyz=0 0.0 0 rpy=0 0 0
- added joint camera2_infra1_optical_joint: type fixed, parent camera2_infra1_frame, child camera2_infra1_optical_frame, origin xyz=0 0 0 rpy=-1.57079632679 0 -1.57079632679
- added joint camera2_infra2_joint: type fixed, parent camera2_link, child camera2_infra2_frame, origin xyz=0 -0.05 0 rpy=0 0 0
- added joint camera2_infra2_optical_joint: type fixed, parent camera2_infra2_frame, child camera2_infra2_optical_frame, origin xyz=0 0 0 rpy=-1.57079632679 0 -1.57079632679
- added joint camera2_joint: type fixed, parent camera_tilt_link, child camera2_bottom_screw_frame, origin xyz=0.041323 -0.023823 0 rpy=3.1416 1.57079632679 1.57079632679, axis 0 0 0
- added joint camera2_link_joint: type fixed, parent camera2_bottom_screw_frame, child camera2_link, origin xyz=0 0.0175 0.0125 rpy=0 0 0
- joint camera_joint: origin xyz=0.041323 -0.023823 0 rpy=3.1416 1.57079632679 1.57079632679 -> xyz=0.29 0 0.13 rpy=3.1416 0 0; parent camera_tilt_link -> base_link

File: boris_description/urdf/boris_description_old.urdf (robot description, URDF)
Before this commit: robot boris_description, 27 links, 26 joints
Links:
- removed link camera2_bottom_screw_frame
- removed link camera2_color_frame
- removed link camera2_color_optical_frame
- removed link camera2_depth_frame
- removed link camera2_depth_optical_frame
- removed link camera2_infra1_frame
- removed link camera2_infra1_optical_frame
- removed link camera2_infra2_frame
- removed link camera2_infra2_optical_frame
- removed link camera2_link
Joints:
- removed joint camera2_color_joint
- removed joint camera2_color_optical_joint
- removed joint camera2_depth_joint
- removed joint camera2_depth_optical_joint
- removed joint camera2_infra1_joint
- removed joint camera2_infra1_optical_joint
- removed joint camera2_infra2_joint
- removed joint camera2_infra2_optical_joint
- removed joint camera2_joint
- removed joint camera2_link_joint
- joint camera_joint: origin xyz=0.304800000000025 0 0.117675 rpy=-1.5707963267949 0 -1.5707963267949 -> xyz=0.041323 -0.023823 0 rpy=3.1416 1.57079632679 1.57079632679; parent base_link -> camera_tilt_link
